Commit message: WIP

File: ros-workspace/src/dr-phil/urdf/dr-phil.urdf.xacro (robot description, xacro)
@@ -3,5 +3,10 @@
   <xacro:include filename="$(find dr-phil)/urdf/common_properties.xacro"/>
   <xacro:include filename="$(find dr-phil)/urdf/dr-phil.gazebo.xacro"/>
-  <link name="base_footprint"/>
+  <xacro:property name="attachment_frame" value="base_footprint"/>
+  <xacro:property name="arm_base_frame" value="base_footprint"/>
+  <xacro:include filename="$(find dr-phil)/urdf/px100.urdf.xacro" />
+  <link name="base_footprint">
+    <child link="" />
+  </link>
   <joint name="base_joint" type="fixed">
     <parent link="base_footprint"/>

Commit message: WIP

File: ros-workspace/src/dr-phil/urdf/dr-phil.urdf.xacro (robot description, xacro)
@@ -39,5 +39,5 @@
       <origin xyz="-0.064 0 0" rpy="0 0 0"/>
       <!-- original value: 1.3729096e+00-->
-      <mass value="1.65e+00"/>
+      <mass value="1.8"/>
       <inertia ixx="8.7002718e-03" ixy="-4.7576583e-05" ixz="1.1160499e-04"
                iyy="8.6195418e-03" iyz="-3.5422299e-06"
