Commit message: integrated px100 arm into urdf

File: ros-workspace/src/dr-phil/urdf/common_properties.xacro (robot description, xacro)
@@ -32,3 +32,6 @@
     <color rgba="1.0 1.0 1.0 1.0"/>
   </material>
+  <material name="interbotix_black">
+    <texture filename="package://dr-phil/meshes/interbotix_black.png"/>
+  </material>
 </robot>

File: ros-workspace/src/dr-phil/urdf/dr-phil.urdf.xacro (robot description, xacro)
@@ -3,6 +3,6 @@
   <xacro:include filename="$(find dr-phil)/urdf/common_properties.xacro"/>
   <xacro:include filename="$(find dr-phil)/urdf/dr-phil.gazebo.xacro"/>
-  <xacro:property name="attachment_frame" value="base_footprint"/>
-  <xacro:property name="arm_base_frame" value="base_footprint"/>
+  <xacro:property name="attachment_frame" value="base_link"/>
+  <xacro:property name="arm_base_frame" value="base_arm"/>
   <xacro:include filename="$(find dr-phil)/urdf/px100.urdf.xacro" />
   <link name="base_footprint">
@@ -22,4 +22,11 @@
       <material name="light_black"/>
     </visual>
+    <visual>
+      <origin xyz="-0.064 0 0.05" rpy="0 0 0"/>
+      <geometry>
+        <mesh filename="package://dr-phil/meshes/bases/waffle_pi_base_layer.stl" scale="0.001 0.001 0.001"/>
+      </geometry>
+      <material name="light_black"/>
+    </visual>
     <collision>
       <origin xyz="-0.064 0 0.047" rpy="0 0 0"/>
@@ -29,6 +36,8 @@
     </collision>
     <inertial>
-      <origin xyz="0 0 0" rpy="0 0 0"/>
-      <mass value="1.3729096e+00"/>
+      <!-- original value: xyz: 0,0,0 -->
+      <origin xyz="-0.064 0 0" rpy="0 0 0"/>
+      <!-- original value: 1.3729096e+00-->
+      <mass value="1.65e+00"/>
       <inertia ixx="8.7002718e-03" ixy="-4.7576583e-05" ixz="1.1160499e-04"
                iyy="8.6195418e-03" iyz="-3.5422299e-06"

File: ros-workspace/src/dr-phil/urdf/px100.urdf.xacro (robot description, xacro)
@@ -13,10 +13,4 @@
   <xacro:arg name="load_gazebo_configs" default="false"/>
   <xacro:property name="pi_offset" value="0.00001"/>
-  <xacro:if value="$(arg load_gazebo_configs)">
-    <xacro:include filename="$(find dr-phil)/config/interbotix_texture.gazebo"/>
-  </xacro:if>
-  <material name="interbotix_black">
-    <texture filename="package://dr-phil/meshes/interbotix_black.png"/>
-  </material>
   <!-- <xacro:if value="$(arg use_world_frame)">
     <link name="world"/>
@@ -27,5 +21,5 @@
   </xacro:if> -->
   <joint name="arm_attachment" type="fixed" >
-    <origin xyz="0 0 0.1" rpy="0 0 0"/>
+    <origin xyz="0.01 0 0.142" rpy="0 0 0"/>
     <parent link="${attachment_frame}"/>
     <child link="$(arg robot_name)/$(arg base_link_frame)"/>
@@ -37,5 +31,5 @@
         <mesh filename="package://dr-phil/meshes/px100_meshes/px100_1_base.stl" scale="0.001 0.001 0.001"/>
       </geometry>
-      <material name="interbotix_black"/>
+      <material name="black"/>
     </visual>
     <collision>
@@ -74,5 +68,5 @@
         <mesh filename="package://dr-phil/meshes/px100_meshes/px100_2_shoulder.stl" scale="0.001 0.001 0.001"/>
       </geometry>
-      <material name="interbotix_black"/>
+      <material name="black"/>
     </visual>
     <collision>
@@ -111,5 +105,5 @@
         <mesh filename="package://dr-phil/meshes/px100_meshes/px100_3_upper_arm.stl" scale="0.001 0.001 0.001"/>
       </geometry>
-      <material name="interbotix_black"/>
+      <material name="black"/>
     </visual>
     <collision>
@@ -148,5 +142,5 @@
         <mesh filename="package://dr-phil/meshes/px100_meshes/px100_4_forearm.stl" scale="0.001 0.001 0.001"/>
       </geometry>
-      <material name="interbotix_black"/>
+      <material name="black"/>
     </visual>
     <collision>
@@ -185,5 +179,5 @@
         <mesh filename="package://dr-phil/meshes/px100_meshes/px100_5_gripper.stl" scale="0.001 0.001 0.001"/>
       </geometry>
-      <material name="interbotix_black"/>
+      <material name="black"/>
     </visual>
     <collision>
@@ -234,5 +228,5 @@
         <mesh filename="package://dr-phil/meshes/px100_meshes/px100_6_gripper_prop.stl" scale="0.001 0.001 0.001"/>
       </geometry>
-      <material name="interbotix_black"/>
+      <material name="black"/>
     </visual>
     <collision>
@@ -262,5 +256,5 @@
           <mesh filename="package://dr-phil/meshes/px100_meshes/px100_9_ar_tag.stl" scale="0.001 0.001 0.001"/>
         </geometry>
-        <material name="interbotix_black"/>
+        <material name="black"/>
       </visual>
       <collision>
@@ -291,5 +285,5 @@
           <mesh filename="package://dr-phil/meshes/px100_meshes/px100_7_gripper_bar.stl" scale="0.001 0.001 0.001"/>
         </geometry>
-        <material name="interbotix_black"/>
+        <material name="black"/>
       </visual>
       <collision>
@@ -342,5 +336,5 @@
             <mesh filename="package://dr-phil/meshes/px100_meshes/px100_8_gripper_finger.stl" scale="0.001 0.001 0.001"/>
           </geometry>
-          <material name="interbotix_black"/>
+          <material name="black"/>
         </visual>
         <collision>
@@ -382,5 +376,5 @@
             <mesh filename="package://dr-phil/meshes/px100_meshes/px100_8_gripper_finger.stl" scale="0.001 0.001 0.001"/>
           </geometry>
-          <material name="interbotix_black"/>
+          <material name="black"/>
         </visual>
         <collision>

Commit message: final adjustments to model

File: ros-workspace/src/dr-phil/urdf/common_properties.xacro (robot description, xacro)
@@ -1,4 +1,19 @@
 <?xml version="1.0" ?>
 <robot name="xacro_properties" xmlns:xacro="http://ros.org/wiki/xacro">
+  <!-- struts for testing lidar collisions -->
+  <xacro:macro name="strut" params="xyz rpy length">
+    <visual>
+      <origin xyz="${xyz}" rpy="${rpy}" />
+      <geometry>
+        <cylinder radius="0.003" length="${length}"/>
+      </geometry>
+    </visual>
+    <collision>
+      <origin xyz="${xyz}" rpy="${rpy}"/>
+      <geometry>
+        <cylinder radius="0.003" length="${length}"/>
+      </geometry>
+    </collision>
+  </xacro:macro>
   <!-- Init colour -->
   <material name="black">

File: ros-workspace/src/dr-phil/urdf/dr-phil.urdf.xacro (robot description, xacro)
@@ -3,9 +3,34 @@
   <xacro:include filename="$(find dr-phil)/urdf/common_properties.xacro"/>
   <xacro:include filename="$(find dr-phil)/urdf/dr-phil.gazebo.xacro"/>
+  <!-- strut measurements -->
+  <xacro:property name="strut_short_length" value="0.035"/>
+  <xacro:property name="strut_long_length" value="0.045"/>
+  <xacro:property name="strut_screw_depth" value="0.0045"/>
+  <xacro:property name="layer_3_strut_length" value="${strut_long_length}"/>
+  <xacro:property name="layer_2_strut_length" value="${strut_long_length}"/>
+  <xacro:property name="layer_1_strut_length" value="${strut_long_length}"/>
+  <xacro:property name="plate_z" value="0.009"/>
+  <xacro:property name="diameter_base" value="0.256"/>
+  <xacro:property name="base_footprint_to_front_strut_plane" value="0.06405"/>
+  <xacro:property name="base_footprint_to_back_strut_plane" value="${diameter_base - base_footprint_to_front_strut_plane}"/>
+  <xacro:property name="base_footprint_to_side_strut_plane" value="0.115"/>
+  <xacro:property name="base_footprint_to_3rd_layer_z" value="0.09140"/>
+  <xacro:property name="base_footprint_to_geometric_centre" value="0.064"/>
+  <xacro:property name="front_to_strut_1" value="0.012"/>
+  <xacro:property name="front_to_strut_2" value="0.024"/>
+  <xacro:property name="side_to_strut_3" value="${diameter_base / 4}"/>
+  <!-- plate measurements -->
+  <xacro:property name="layer_3_z" value="${(plate_z * 2) + (layer_1_strut_length + layer_2_strut_length + layer_3_strut_length) - (2 * 2 * strut_screw_depth)}"/>
+  <!-- arm measurements -->
+  <xacro:property name="px100_from_centre_to_back_box" value="0.04678"/>
+  <xacro:property name="px100_back_box_width" value="0.08107"/>
   <xacro:property name="attachment_frame" value="base_link"/>
+  <xacro:property name="arm_origin">
+      <origin xyz="${-base_footprint_to_geometric_centre + px100_from_centre_to_back_box + (px100_back_box_width / 2)} 0 ${layer_3_z + plate_z}" rpy="0 0 0"/>
+  </xacro:property>
   <xacro:property name="arm_base_frame" value="base_arm"/>
   <xacro:include filename="$(find dr-phil)/urdf/px100.urdf.xacro" />
+  <!-- dr-phil -->
   <link name="base_footprint">
-    <child link="" />
   </link>
   <joint name="base_joint" type="fixed">
@@ -22,6 +47,7 @@
       <material name="light_black"/>
     </visual>
-    <visual>
-      <origin xyz="-0.064 0 0.05" rpy="0 0 0"/>
+    <!-- 3rd layer -->
+    <visual>
+      <origin xyz="-0.064 0 ${layer_3_z}" rpy="0 0 0"/>
       <geometry>
         <mesh filename="package://dr-phil/meshes/bases/waffle_pi_base_layer.stl" scale="0.001 0.001 0.001"/>
@@ -29,10 +55,20 @@
       <material name="light_black"/>
     </visual>
-    <collision>
-      <origin xyz="-0.064 0 0.047" rpy="0 0 0"/>
-      <geometry>
-        <box size="0.266 0.266 0.094"/>
-      </geometry>
-    </collision>
+    <!-- strut 1 - front left -->
+    <xacro:strut xyz="${base_footprint_to_front_strut_plane} ${front_to_strut_1} ${base_footprint_to_3rd_layer_z + (layer_3_strut_length/2)}" rpy="0 0 0" length="${layer_3_strut_length}"/>
+    <!-- strut 2 - front right -->
+    <xacro:strut xyz="${base_footprint_to_front_strut_plane} ${-front_to_strut_2} ${base_footprint_to_3rd_layer_z + (layer_3_strut_length/2)}" rpy="0 0 0" length="${layer_3_strut_length}"/>
+    <!-- strut 3 - right side front -->
+    <xacro:strut xyz="${-base_footprint_to_geometric_centre + side_to_strut_3} ${-base_footprint_to_side_strut_plane} ${base_footprint_to_3rd_layer_z + (layer_3_strut_length/2)}" rpy="0 0 0" length="${layer_3_strut_length}"/>
+    <!-- strut 4 - right side back -->
+    <xacro:strut xyz="${-base_footprint_to_geometric_centre - side_to_strut_3} ${-base_footprint_to_side_strut_plane} ${base_footprint_to_3rd_layer_z + (layer_3_strut_length/2)}" rpy="0 0 0" length="${layer_3_strut_length}"/>
+    <!-- strut 5 - back right -->
+    <xacro:strut xyz="${-base_footprint_to_back_strut_plane} ${-front_to_strut_1} ${base_footprint_to_3rd_layer_z + (layer_3_strut_length/2)}" rpy="0 0 0" length="${layer_3_strut_length}"/>
+    <!-- strut 6 - back left -->
+    <xacro:strut xyz="${-base_footprint_to_back_strut_plane} ${front_to_strut_2} ${base_footprint_to_3rd_layer_z + (layer_3_strut_length/2)}" rpy="0 0 0" length="${layer_3_strut_length}"/>
+    <!-- strut 7 - left side front -->
+    <xacro:strut xyz="${-base_footprint_to_geometric_centre + side_to_strut_3} ${base_footprint_to_side_strut_plane} ${base_footprint_to_3rd_layer_z + (layer_3_strut_length/2)}" rpy="0 0 0" length="${layer_3_strut_length}"/>
+    <!-- strut 8 - left side back -->
+    <xacro:strut xyz="${-base_footprint_to_geometric_centre - side_to_strut_3} ${base_footprint_to_side_strut_plane} ${base_footprint_to_3rd_layer_z + (layer_3_strut_length/2)}" rpy="0 0 0" length="${layer_3_strut_length}"/>
     <inertial>
       <!-- original value: xyz: 0,0,0 -->

File: ros-workspace/src/dr-phil/urdf/px100.urdf.xacro (robot description, xacro)
@@ -13,13 +13,6 @@
   <xacro:arg name="load_gazebo_configs" default="false"/>
   <xacro:property name="pi_offset" value="0.00001"/>
-  <!-- <xacro:if value="$(arg use_world_frame)">
-    <link name="world"/>
-    <joint name="fixed" type="fixed">
-      <parent link="world"/>
-      <child link="$(arg robot_name)/$(arg base_link_frame)"/>
-    </joint>
-  </xacro:if> -->
   <joint name="arm_attachment" type="fixed" >
-    <origin xyz="0.01 0 0.142" rpy="0 0 0"/>
+    <xacro:insert_block name="arm_origin" />
     <parent link="${attachment_frame}"/>
     <child link="$(arg robot_name)/$(arg base_link_frame)"/>
