Commit message: Added bottle
Added the bottle, lid and and base plate to hold the bottle

File: ros-workspace/src/dr_phil_description/urdf/dr-phil.urdf.xacro (robot description, xacro)
@@ -81,4 +81,76 @@
     </inertial>
   </link>
+  <joint name="bottle_base_joint" type="fixed">
+    <parent link="base_link"/>
+    <child link="bottle_base_link" />
+    <origin xyz="0 0 0.010" rpy="0 0 0"/>
+  </joint>
+  <link name="bottle_base_link">
+    <visual>
+      <origin xyz="-0.088 -0.028 ${layer_3_z-0.0075}" rpy="0 0 0"/>
+      <geometry>
+        <mesh filename="package://dr_phil_description/meshes/spray_components/bottle_base.stl" scale="0.001 0.001 0.001"/>
+      </geometry>
+    </visual>
+    <collision>
+      <origin xyz="-0.088 -0.028 ${layer_3_z-0.0075}" rpy="0 0 0"/>
+      <geometry>
+        <mesh filename="package://dr_phil_description/meshes/spray_components/bottle_base.stl" scale="0.001 0.001 0.001"/>
+      </geometry>
+    </collision>
+    <inertial>
+      <origin xyz="-0.088 -0.028 ${layer_3_z-0.0075}" rpy="0 0 0"/>
+      <mass value="0.036"/>
+      <inertia ixx="0.00" iyy="0.00" izz="0.000" ixy="0.0000000000" ixz="0.0000000000" iyz="0" />
+    </inertial>
+  </link>
+  <joint name="bottle_joint" type="fixed">
+    <parent link="bottle_base_link"/>
+    <child link="bottle_link" />
+    <origin xyz="0 0 0.010" rpy="0 0 0"/>
+  </joint>
+  <link name="bottle_link">
+    <visual>
+      <origin xyz="-0.1695 -0.0965 ${layer_3_z}" rpy="0 0 ${pi/2}"/>
+      <geometry>
+        <mesh filename="package://dr_phil_description/meshes/spray_components/bottle_reduced_resized.stl" scale="0.001 0.001 0.001"/>
+      </geometry>
+    </visual>
+    <collision>
+      <origin xyz="-0.1695 -0.0965 ${layer_3_z}" rpy="0 0 ${pi/2}"/>
+      <geometry>
+        <mesh filename="package://dr_phil_description/meshes/spray_components/bottle_reduced_resized.stl" scale="0.001 0.001 0.001"/>
+      </geometry>
+    </collision>
+    <inertial>
+      <origin xyz="-0.1695 -0.0965 ${layer_3_z}" rpy="0 0 0"/>
+      <mass value="0.074"/>
+      <inertia ixx="0.00" iyy="0.00" izz="0.000" ixy="0.0000000000" ixz="0.0000000000" iyz="0" />
+    </inertial>
+  </link>
+  <joint name="bottle_cap_joint" type="fixed">
+    <parent link="bottle_base_link"/>
+    <child link="bottle_cap_link" />
+    <origin xyz="0 0 0.010" rpy="0 0 0"/>
+  </joint>
+  <link name="bottle_cap_link">
+    <visual>
+      <origin xyz="-0.1519 -0.06 ${layer_3_z+0.096}" rpy="${pi} 0 0"/>
+      <geometry>
+        <mesh filename="package://dr_phil_description/meshes/spray_components/bottle_lid.stl" scale="0.001 0.001 0.001"/>
+      </geometry>
+    </visual>
+    <collision>
+      <origin xyz="-0.1519 -0.06 ${layer_3_z+0.096}" rpy="${pi} 0 0"/>
+      <geometry>
+        <mesh filename="package://dr_phil_description/meshes/spray_components/bottle_lid.stl" scale="0.001 0.001 0.001"/>
+      </geometry>
+    </collision>
+    <inertial>
+      <origin xyz="-0.1519 -0.06 ${layer_3_z+0.096}" rpy="0 0 0"/>
+      <mass value="0.016"/>
+      <inertia ixx="0.00" iyy="0.00" izz="0.000" ixy="0.0000000000" ixz="0.0000000000" iyz="0" />
+    </inertial>
+  </link>
   <joint name="wheel_left_joint" type="continuous">
     <parent link="base_link"/>

Commit message: Point cloud generator of sanitation area
Added a point cloud generator for area within range of the spray. Added seperate node to save to file just the part of the cloud surrounding the handle. Rearranged position of pump and tank on model to match irl setup.

File: ros-workspace/src/dr_phil_description/urdf/dr-phil.urdf.xacro (robot description, xacro)
@@ -88,5 +88,5 @@
   <link name="bottle_base_link">
     <visual>
-      <origin xyz="-0.088 -0.028 ${layer_3_z-0.0075}" rpy="0 0 0"/>
+      <origin xyz="-0.088 0.028 ${layer_3_z-0.0075}" rpy="0 0 ${-pi/2}"/>
       <geometry>
         <mesh filename="package://dr_phil_description/meshes/spray_components/bottle_base.stl" scale="0.001 0.001 0.001"/>
@@ -94,5 +94,5 @@
     </visual>
     <collision>
-      <origin xyz="-0.088 -0.028 ${layer_3_z-0.0075}" rpy="0 0 0"/>
+      <origin xyz="-0.088 -0.028 ${layer_3_z-0.0075}" rpy="0 0 ${-pi/2}"/>
       <geometry>
         <mesh filename="package://dr_phil_description/meshes/spray_components/bottle_base.stl" scale="0.001 0.001 0.001"/>
@@ -100,5 +100,5 @@
     </collision>
     <inertial>
-      <origin xyz="-0.088 -0.028 ${layer_3_z-0.0075}" rpy="0 0 0"/>
+      <origin xyz="-0.088 0.028 ${layer_3_z-0.0075}" rpy="0 0 ${-pi/2}"/>
       <mass value="0.036"/>
       <inertia ixx="0.00" iyy="0.00" izz="0.000" ixy="0.0000000000" ixz="0.0000000000" iyz="0" />
@@ -112,5 +112,5 @@
   <link name="bottle_link">
     <visual>
-      <origin xyz="-0.1695 -0.0965 ${layer_3_z}" rpy="0 0 ${pi/2}"/>
+      <origin xyz="-0.156 0.1095 ${layer_3_z}" rpy="0 0 0"/>
       <geometry>
         <mesh filename="package://dr_phil_description/meshes/spray_components/bottle_reduced_resized.stl" scale="0.001 0.001 0.001"/>
@@ -118,5 +118,5 @@
     </visual>
     <collision>
-      <origin xyz="-0.1695 -0.0965 ${layer_3_z}" rpy="0 0 ${pi/2}"/>
+      <origin xyz="-0.156 0.1095 ${layer_3_z}" rpy="0 0 0"/>
       <geometry>
         <mesh filename="package://dr_phil_description/meshes/spray_components/bottle_reduced_resized.stl" scale="0.001 0.001 0.001"/>
@@ -124,5 +124,5 @@
     </collision>
     <inertial>
-      <origin xyz="-0.1695 -0.0965 ${layer_3_z}" rpy="0 0 0"/>
+      <origin xyz="-0.156 0.1095 ${layer_3_z}" rpy="0 0 0"/>
       <mass value="0.074"/>
       <inertia ixx="0.00" iyy="0.00" izz="0.000" ixy="0.0000000000" ixz="0.0000000000" iyz="0" />
@@ -136,5 +136,5 @@
   <link name="bottle_cap_link">
     <visual>
-      <origin xyz="-0.1519 -0.06 ${layer_3_z+0.096}" rpy="${pi} 0 0"/>
+      <origin xyz="-0.1289 0.101 ${layer_3_z+0.096}" rpy="${pi} 0 0"/>
       <geometry>
         <mesh filename="package://dr_phil_description/meshes/spray_components/bottle_lid.stl" scale="0.001 0.001 0.001"/>
@@ -150,4 +150,52 @@
       <origin xyz="-0.1519 -0.06 ${layer_3_z+0.096}" rpy="0 0 0"/>
       <mass value="0.016"/>
+      <inertia ixx="0.00" iyy="0.00" izz="0.000" ixy="0.0000000000" ixz="0.0000000000" iyz="0" />
+    </inertial>
+  </link>
+  <joint name="pump_joint" type="fixed">
+    <parent link="bottle_base_link"/>
+    <child link="pump_link" />
+    <origin xyz="0 0 0.010" rpy="0 0 0"/>
+  </joint>
+  <link name="pump_link">
+    <visual>
+      <origin xyz="-0.14 -0.07  ${layer_3_z-0.011}" rpy="0 0 ${pi}"/>
+      <geometry>
+        <mesh filename="package://dr_phil_description/meshes/spray_components/pump_w_bracket_tinker.stl" scale="0.001 0.001 0.001"/>
+      </geometry>
+    </visual>
+    <collision>
+      <origin xyz="-0.088 -0.028 ${layer_3_z}" rpy="0 0 0"/>
+      <geometry>
+        <mesh filename="package://dr_phil_description/meshes/spray_components/pump_w_bracket_tinker.stl" scale="0.001 0.001 0.001"/>
+      </geometry>
+    </collision>
+    <inertial>
+      <origin xyz="-0.088 -0.028 ${layer_3_z}" rpy="0 0 0"/>
+      <mass value="0.036"/>
+      <inertia ixx="0.00" iyy="0.00" izz="0.000" ixy="0.0000000000" ixz="0.0000000000" iyz="0" />
+    </inertial>
+  </link>
+  <joint name="pump_dummy_joint" type="fixed">
+    <parent link="bottle_base_link"/>
+    <child link="pump_dummy_link" />
+    <origin xyz="0 0 0.010" rpy="0 0 0"/>
+  </joint>
+  <link name="pump_dummy_link">
+    <visual>
+      <origin xyz="-0.101 -0.07  ${layer_3_z+0.014}" rpy="0 0 ${pi}"/>
+      <geometry>
+        <mesh filename="package://dr_phil_description/meshes/spray_components/12V Diaphragm Pump RS-385 - NO BRACKETS v1.stl" scale="0.001 0.001 0.001"/>
+      </geometry>
+    </visual>
+    <collision>
+      <origin xyz="-0.088 -0.028 ${layer_3_z}" rpy="0 0 0"/>
+      <geometry>
+        <mesh filename="package://dr_phil_description/meshes/spray_components/12V Diaphragm Pump RS-385 - NO BRACKETS v1.stl" scale="0.001 0.001 0.001"/>
+      </geometry>
+    </collision>
+    <inertial>
+      <origin xyz="-0.088 -0.028 ${layer_3_z}" rpy="0 0 0"/>
+      <mass value="0.036"/>
       <inertia ixx="0.00" iyy="0.00" izz="0.000" ixy="0.0000000000" ixz="0.0000000000" iyz="0" />
     </inertial>

File: ros-workspace/src/dr_phil_description/urdf/px100.urdf.xacro (robot description, xacro)
@@ -230,4 +230,54 @@
     </inertial>
   </link>
+  <joint name="$(arg robot_name)/led_joint1" type="fixed">
+  <origin xyz="0.044 0.019 0.0345" rpy="${-pi/2} 0 ${-pi/2}"/>
+  <parent link="$(arg robot_name)/gripper_link"/>
+  <child link="$(arg robot_name)/led_link1"/> </joint>
+<link name="$(arg robot_name)/led_link1">
+  </link>
+    <gazebo reference="$(arg robot_name)/gripper_link">
+    <sensor type="depth" name="depth_camera">
+    <pose>0.06645 0 0.043 0 0 0</pose>
+      <update_rate>1</update_rate>
+      <camera>
+        <horizontal_fov>${pi/6}</horizontal_fov>
+        <image>
+          <width>640</width>
+          <height>480</height>
+          <format>R8G8B8</format>
+        </image>
+        <clip>
+          <near>0.02</near>
+          <far>1</far>
+        </clip>
+      </camera>
+          <plugin name="camera_plugin" filename="libgazebo_ros_openni_kinect.so">
+          <baseline>0.2</baseline>
+          <alwaysOn>true</alwaysOn>
+          <!-- Keep this zero, update_rate in the parent <sensor> tag
+            will control the frame rate. -->
+          <updateRate>0.0</updateRate>
+          <cameraName>depth_camera</cameraName>
+          <imageTopicName>/depth_camera/color/image_raw</imageTopicName>
+          <cameraInfoTopicName>/depth_camera/color/camera_info</cameraInfoTopicName>
+          <depthImageTopicName>/depth_camera/depth/image_raw</depthImageTopicName>
+          <depthImageCameraInfoTopicName>/depth_camera/depth/camera_info</depthImageCameraInfoTopicName>
+          <pointCloudTopicName>/depth_camera/depth/points</pointCloudTopicName>
+          <frameName>odom</frameName>
+          <pointCloudCutoff>0.0</pointCloudCutoff>
+          <pointCloudCutoffMax>1.0</pointCloudCutoffMax>
+          <distortionK1>0</distortionK1>
+          <distortionK2>0</distortionK2>
+          <distortionK3>0</distortionK3>
+          <distortionT1>0</distortionT1>
+          <distortionT2>0</distortionT2>
+          <CxPrime>0</CxPrime>
+          <Cx>0</Cx>
+          <Cy>0</Cy>
+          <focalLength>0</focalLength>
+          <hackBaseline>0</hackBaseline>
+        </plugin>
+    </sensor>
+  </gazebo>
   <gazebo reference="$(arg robot_name)/gripper_link">
   <light name ='led' type = 'spot'>

Commit message: changed moveit setup and costmap parameters

File: ros-workspace/src/dr_phil_description/urdf/dr-phil.urdf.xacro (robot description, xacro)
@@ -73,7 +73,7 @@
     <inertial>
       <!-- original value: xyz: 0,0,0 -->
-      <origin xyz="-0.064 0 0" rpy="0 0 0"/>
+      <origin xyz="-0.05 0 0" rpy="0 0 0"/>
       <!-- original value: 1.3729096e+00-->
-      <mass value="1.8"/>
+      <mass value="1.3729096e+00"/>
       <inertia ixx="8.7002718e-03" ixy="-4.7576583e-05" ixz="1.1160499e-04"
                iyy="8.6195418e-03" iyz="-3.5422299e-06"

File: ros-workspace/src/dr_phil_description/urdf/px100.urdf.xacro (robot description, xacro)
@@ -40,4 +40,5 @@
     </collision>
     <inertial>
+                                      <!--- original value x:0.0332053000 -->
       <origin rpy="0 0 ${pi/2}" xyz="-0.0332053000 0.0008915770 0.0211913000"/>
       <mass value="0.395887" />

Commit message: changed weight of bottle to stop robot from tipping when arm extended

File: ros-workspace/src/dr_phil_description/urdf/dr-phil.urdf.xacro (robot description, xacro)
@@ -75,5 +75,5 @@
       <origin xyz="-0.05 0 0" rpy="0 0 0"/>
       <!-- original value: 1.3729096e+00-->
-      <mass value="1.3729096e+00"/>
+      <mass value="1.6729096e+00"/>
       <inertia ixx="8.7002718e-03" ixy="-4.7576583e-05" ixz="1.1160499e-04"
                iyy="8.6195418e-03" iyz="-3.5422299e-06"
@@ -125,5 +125,5 @@
     <inertial>
       <origin xyz="-0.1695 -0.0965 ${layer_3_z}" rpy="0 0 0"/>
-      <mass value="0.074"/>
+      <mass value="0.1"/>
       <inertia ixx="0.00" iyy="0.00" izz="0.000" ixy="0.0000000000" ixz="0.0000000000" iyz="0" />
     </inertial>

Commit message: added pump to model

File: ros-workspace/src/dr_phil_description/urdf/dr-phil.urdf.xacro (robot description, xacro)
@@ -88,5 +88,5 @@
   <link name="bottle_base_link">
     <visual>
-      <origin xyz="-0.088 -0.028 ${layer_3_z-0.0075}" rpy="0 0 0"/>
+      <origin xyz="-0.088 0.028 ${layer_3_z-0.0075}" rpy="0 0 ${-pi/2}"/>
       <geometry>
         <mesh filename="package://dr_phil_description/meshes/spray_components/bottle_base.stl" scale="0.001 0.001 0.001"/>
@@ -94,5 +94,5 @@
     </visual>
     <collision>
-      <origin xyz="-0.088 -0.028 ${layer_3_z-0.0075}" rpy="0 0 0"/>
+      <origin xyz="-0.088 -0.028 ${layer_3_z-0.0075}" rpy="0 0 ${-pi/2}"/>
       <geometry>
         <mesh filename="package://dr_phil_description/meshes/spray_components/bottle_base.stl" scale="0.001 0.001 0.001"/>
@@ -100,5 +100,5 @@
     </collision>
     <inertial>
-      <origin xyz="-0.088 -0.028 ${layer_3_z-0.0075}" rpy="0 0 0"/>
+      <origin xyz="-0.088 0.028 ${layer_3_z-0.0075}" rpy="0 0 ${-pi/2}"/>
       <mass value="0.036"/>
       <inertia ixx="0.00" iyy="0.00" izz="0.000" ixy="0.0000000000" ixz="0.0000000000" iyz="0" />
@@ -112,5 +112,5 @@
   <link name="bottle_link">
     <visual>
-      <origin xyz="-0.1695 -0.0965 ${layer_3_z}" rpy="0 0 ${pi/2}"/>
+      <origin xyz="-0.156 0.1095 ${layer_3_z}" rpy="0 0 0"/>
       <geometry>
         <mesh filename="package://dr_phil_description/meshes/spray_components/bottle_reduced_resized.stl" scale="0.001 0.001 0.001"/>
@@ -118,5 +118,5 @@
     </visual>
     <collision>
-      <origin xyz="-0.1695 -0.0965 ${layer_3_z}" rpy="0 0 ${pi/2}"/>
+      <origin xyz="-0.156 0.1095 ${layer_3_z}" rpy="0 0 0"/>
       <geometry>
         <mesh filename="package://dr_phil_description/meshes/spray_components/bottle_reduced_resized.stl" scale="0.001 0.001 0.001"/>
@@ -124,6 +124,6 @@
     </collision>
     <inertial>
-      <origin xyz="-0.1695 -0.0965 ${layer_3_z}" rpy="0 0 0"/>
-      <mass value="0.1"/>
+      <origin xyz="-0.156 0.1095 ${layer_3_z}" rpy="0 0 0"/>
+      <mass value="0.074"/>
       <inertia ixx="0.00" iyy="0.00" izz="0.000" ixy="0.0000000000" ixz="0.0000000000" iyz="0" />
     </inertial>
@@ -136,5 +136,5 @@
   <link name="bottle_cap_link">
     <visual>
-      <origin xyz="-0.1519 -0.06 ${layer_3_z+0.096}" rpy="${pi} 0 0"/>
+      <origin xyz="-0.1289 0.101 ${layer_3_z+0.096}" rpy="${pi} 0 0"/>
       <geometry>
         <mesh filename="package://dr_phil_description/meshes/spray_components/bottle_lid.stl" scale="0.001 0.001 0.001"/>
@@ -150,4 +150,52 @@
       <origin xyz="-0.1519 -0.06 ${layer_3_z+0.096}" rpy="0 0 0"/>
       <mass value="0.016"/>
+      <inertia ixx="0.00" iyy="0.00" izz="0.000" ixy="0.0000000000" ixz="0.0000000000" iyz="0" />
+    </inertial>
+  </link>
+  <joint name="pump_joint" type="fixed">
+    <parent link="bottle_base_link"/>
+    <child link="pump_link" />
+    <origin xyz="0 0 0.010" rpy="0 0 0"/>
+  </joint>
+  <link name="pump_link">
+    <visual>
+      <origin xyz="-0.14 -0.07  ${layer_3_z-0.011}" rpy="0 0 ${pi}"/>
+      <geometry>
+        <mesh filename="package://dr_phil_description/meshes/spray_components/pump_w_bracket_tinker.stl" scale="0.001 0.001 0.001"/>
+      </geometry>
+    </visual>
+    <collision>
+      <origin xyz="-0.088 -0.028 ${layer_3_z}" rpy="0 0 0"/>
+      <geometry>
+        <mesh filename="package://dr_phil_description/meshes/spray_components/pump_w_bracket_tinker.stl" scale="0.001 0.001 0.001"/>
+      </geometry>
+    </collision>
+    <inertial>
+      <origin xyz="-0.088 -0.028 ${layer_3_z}" rpy="0 0 0"/>
+      <mass value="0.036"/>
+      <inertia ixx="0.00" iyy="0.00" izz="0.000" ixy="0.0000000000" ixz="0.0000000000" iyz="0" />
+    </inertial>
+  </link>
+  <joint name="pump_dummy_joint" type="fixed">
+    <parent link="bottle_base_link"/>
+    <child link="pump_dummy_link" />
+    <origin xyz="0 0 0.010" rpy="0 0 0"/>
+  </joint>
+  <link name="pump_dummy_link">
+    <visual>
+      <origin xyz="-0.101 -0.07  ${layer_3_z+0.014}" rpy="0 0 ${pi}"/>
+      <geometry>
+        <mesh filename="package://dr_phil_description/meshes/spray_components/12V Diaphragm Pump RS-385 - NO BRACKETS v1.stl" scale="0.001 0.001 0.001"/>
+      </geometry>
+    </visual>
+    <collision>
+      <origin xyz="-0.088 -0.028 ${layer_3_z}" rpy="0 0 0"/>
+      <geometry>
+        <mesh filename="package://dr_phil_description/meshes/spray_components/12V Diaphragm Pump RS-385 - NO BRACKETS v1.stl" scale="0.001 0.001 0.001"/>
+      </geometry>
+    </collision>
+    <inertial>
+      <origin xyz="-0.088 -0.028 ${layer_3_z}" rpy="0 0 0"/>
+      <mass value="0.036"/>
       <inertia ixx="0.00" iyy="0.00" izz="0.000" ixy="0.0000000000" ixz="0.0000000000" iyz="0" />
     </inertial>
