Commit message: Added nozzle with controllable light
Added the nozzle to the end of the arm, with a light source to simulate spraying. use  rostopic pub /spray_controller/command std_msgs/Float32 '1'
 for on, 0 for off

File: ros-workspace/src/dr_phil_description/urdf/px100.urdf.xacro (robot description, xacro)
@@ -206,4 +206,44 @@
     <dynamics friction="0.1"/>
   </joint>
+  <joint name="$(arg robot_name)/led_joint" type="fixed">
+  <origin xyz="0.044 0.019 0.0345" rpy="0 0 0"/>
+  <parent link="$(arg robot_name)/gripper_link"/>
+  <child link="$(arg robot_name)/led_link"/> </joint>
+<link name="$(arg robot_name)/led_link">
+   <visual>
+      <origin rpy="0 0 0" xyz="0 0.0 0.0"/>
+      <geometry>
+        <mesh filename="package://dr_phil_description/meshes/spray_components/8_5mm_nozzle.stl" scale="0.001 0.001 0.001"/>
+      </geometry>
+      <material name="black"/>
+    </visual>
+   <collision>
+      <origin rpy="0 0 0" xyz="0 0 0"/>
+      <geometry>
+        <mesh filename="package://dr_phil_description/meshes/spray_components/8_5mm_nozzle.stl" scale="0.001 0.001 0.001"/>
+      </geometry>
+    </collision>
+    <inertial>
+      <origin rpy="0 0 0" xyz="0 0 0"/>
+      <mass value="0.002" />
+      <inertia ixx="0.00" iyy="0.00" izz="0.000" ixy="0.0000000000" ixz="0.0000000000" iyz="0" />
+    </inertial>
+  </link>
+  <gazebo reference="$(arg robot_name)/gripper_link">
+  <light name ='led' type = 'spot'>
+    <pose>0.06645 0 0.043 0 ${-pi/2} 0</pose><!--you can place light position here ,and it is useless to give position in link-->
+    <attenuation>
+            <range>1</range>
+          </attenuation>
+          <diffuse>1 1 1 0</diffuse>
+          <specular>1 1 1 0</specular>
+          <spot>
+            <inner_angle>${pi/6}</inner_angle>
+            <outer_angle>${pi/6}</outer_angle>
+            <falloff>1</falloff>
+          </spot>
+          <cast_shadows>1</cast_shadows>
+  </light>
+  </gazebo>
   <transmission name="trans_gripper">
     <type>transmission_interface/SimpleTransmission</type>

Commit message: changed urdf description

File: ros-workspace/src/dr_phil_description/urdf/px100.urdf.xacro (robot description, xacro)
@@ -3,4 +3,5 @@
   <gazebo>
     <plugin name="gazebo_ros_control" filename="libgazebo_ros_control.so">
+      <robotNamespace>/</robotNamespace>
     </plugin>
   </gazebo>
@@ -38,5 +39,6 @@
     </inertial>
   </link>
-  <joint name="waist" type="revolute">
+  <!-- joint 1 -->
+  <joint name="joint1" type="revolute">
     <axis xyz="0 0 1"/>
     <limit effort="1" lower="${-pi + pi_offset}" upper="${pi - pi_offset}" velocity="${pi}"/>
@@ -46,10 +48,10 @@
     <dynamics friction="0.1"/>
   </joint>
-  <transmission name="trans_waist">
+  <transmission name="trans_joint1">
     <type>transmission_interface/SimpleTransmission</type>
-    <joint name="waist">
-      <hardwareInterface>hardware_interface/EffortJointInterface</hardwareInterface>
-    </joint>
-    <actuator name="waist_motor">
+    <joint name="joint1">
+        <hardwareInterface>hardware_interface/PositionJointInterface</hardwareInterface>
+    </joint>
+    <actuator name="motor1">
       <mechanicalReduction>1</mechanicalReduction>
     </actuator>
@@ -75,5 +77,6 @@
     </inertial>
   </link>
-  <joint name="shoulder" type="revolute">
+  <!-- joint2 -->
+  <joint name="joint2" type="revolute">
     <axis xyz="0 1 0"/>
     <limit effort="2" lower="${radians(-111)}" upper="${radians(107)}" velocity="${pi}"/>
@@ -83,10 +86,10 @@
     <dynamics friction="0.1"/>
   </joint>
-  <transmission name="trans_shoulder">
+  <transmission name="trans_joint2">
     <type>transmission_interface/SimpleTransmission</type>
-    <joint name="shoulder">
-      <hardwareInterface>hardware_interface/EffortJointInterface</hardwareInterface>
-    </joint>
-    <actuator name="shoulder_motor">
+    <joint name="joint2">
+        <hardwareInterface>hardware_interface/PositionJointInterface</hardwareInterface>
+    </joint>
+    <actuator name="motor2">
       <mechanicalReduction>1</mechanicalReduction>
     </actuator>
@@ -112,5 +115,6 @@
     </inertial>
   </link>
-  <joint name="elbow" type="revolute">
+  <!-- joint3 -->
+  <joint name="joint3" type="revolute">
     <axis xyz="0 1 0"/>
     <limit effort="2" lower="${radians(-121)}" upper="${radians(92)}" velocity="${pi}"/>
@@ -120,10 +124,10 @@
     <dynamics friction="0.1"/>
   </joint>
-  <transmission name="trans_elbow">
+  <transmission name="trans_joint3">
     <type>transmission_interface/SimpleTransmission</type>
-    <joint name="elbow">
-      <hardwareInterface>hardware_interface/EffortJointInterface</hardwareInterface>
-    </joint>
-    <actuator name="elbow_motor">
+    <joint name="joint3">
+        <hardwareInterface>hardware_interface/PositionJointInterface</hardwareInterface>
+    </joint>
+    <actuator name="motor3">
       <mechanicalReduction>1</mechanicalReduction>
     </actuator>
@@ -149,5 +153,6 @@
     </inertial>
   </link>
-  <joint name="wrist_angle" type="revolute">
+  <!-- joint4 -->
+  <joint name="joint4" type="revolute">
     <axis xyz="0 1 0"/>
     <limit effort="1" lower="${radians(-100)}" upper="${radians(123)}"  velocity="${pi}"/>
@@ -157,13 +162,14 @@
     <dynamics friction="0.1"/>
   </joint>
-  <transmission name="trans_wrist_angle">
+  <transmission name="trans_joint4">
     <type>transmission_interface/SimpleTransmission</type>
-    <joint name="wrist_angle">
-      <hardwareInterface>hardware_interface/EffortJointInterface</hardwareInterface>
-    </joint>
-    <actuator name="wrist_angle_motor">
+    <joint name="joint4">
+        <hardwareInterface>hardware_interface/PositionJointInterface</hardwareInterface>
+    </joint>
+    <actuator name="motor4">
       <mechanicalReduction>1</mechanicalReduction>
     </actuator>
   </transmission>
+  <!-- gripper link -->
   <link name="$(arg robot_name)/gripper_link">
     <visual>
@@ -198,5 +204,6 @@
     </inertial>
   </link>
-  <joint name="gripper" type="continuous">
+  <!-- gripper -->
+  <joint name="gripper_spindle" type="continuous">
     <axis xyz="1 0 0"/>
     <limit effort="1" velocity="${pi}"/>
@@ -208,8 +215,8 @@
   <transmission name="trans_gripper">
     <type>transmission_interface/SimpleTransmission</type>
-    <joint name="gripper">
+    <joint name="gripper_spindle">
       <hardwareInterface>hardware_interface/EffortJointInterface</hardwareInterface>
     </joint>
-    <actuator name="gripper_motor">
+    <actuator name="gripper_spindle_motor">
       <mechanicalReduction>1</mechanicalReduction>
     </actuator>
@@ -306,5 +313,5 @@
     <!-- If the gripper fingers are being used, add those as well -->
     <xacro:if value="$(arg show_gripper_fingers)">
-      <joint name="left_finger" type="prismatic">
+      <joint name="gripper" type="prismatic">
         <axis xyz="0 1 0"/>
         <limit effort="5" lower="0.015" upper="0.037" velocity="1"/>
@@ -314,10 +321,10 @@
         <dynamics friction="0.1"/>
       </joint>
-      <transmission name="trans_left_finger">
+      <transmission name="trans_gripper">
         <type>transmission_interface/SimpleTransmission</type>
-        <joint name="left_finger">
+        <joint name="gripper">
           <hardwareInterface>hardware_interface/EffortJointInterface</hardwareInterface>
         </joint>
-        <actuator name="left_finger_motor">
+        <actuator name="motor_gripper">
           <mechanicalReduction>1</mechanicalReduction>
         </actuator>
@@ -343,5 +350,5 @@
         </inertial>
       </link>
-      <joint name="right_finger" type="prismatic">
+      <joint name="gripper_sub" type="prismatic">
         <axis xyz="0 1 0"/>
         <limit effort="5" lower="-0.037" upper="-0.015" velocity="1"/>
@@ -350,14 +357,12 @@
         <child link="$(arg robot_name)/right_finger_link"/>
         <dynamics friction="0.1"/>
-        <xacro:unless value="$(arg load_gazebo_configs)">
-          <mimic joint="left_finger" multiplier="-1" offset="0"/>
-        </xacro:unless>
+        <mimic joint="gripper" multiplier="-1" offset="0"/>
       </joint>
-      <transmission name="trans_right_finger">
+      <transmission name="trans_gripper_sub">
         <type>transmission_interface/SimpleTransmission</type>
-        <joint name="right_finger">
+        <joint name="gripper_sub">
           <hardwareInterface>hardware_interface/EffortJointInterface</hardwareInterface>
         </joint>
-        <actuator name="right_finger_motor">
+        <actuator name="motor_gripper_sub">
           <mechanicalReduction>1</mechanicalReduction>
         </actuator>

Commit message: fixed mimic joint functionality in gazebo not working

File: ros-workspace/src/dr_phil_description/urdf/px100.urdf.xacro (robot description, xacro)
@@ -4,4 +4,10 @@
     <plugin name="gazebo_ros_control" filename="libgazebo_ros_control.so">
       <robotNamespace>/</robotNamespace>
+    </plugin>
+    <plugin name="libroboticsgroup_gazebo_mimic_joint_plugin" filename="libroboticsgroup_gazebo_mimic_joint_plugin.so">
+      <joint>gripper</joint>
+      <mimicJoint>gripper_sub</mimicJoint>
+      <multiplier>-1</multiplier>
+      <has_pid>true</has_pid>
     </plugin>
   </gazebo>

Commit message: added coverage visualisation

File: ros-workspace/src/dr_phil_description/urdf/px100.urdf.xacro (robot description, xacro)
@@ -244,4 +244,54 @@
     </inertial>
   </link>
+    <joint name="$(arg robot_name)/led_joint1" type="fixed">
+  <origin xyz="0.044 0.019 0.0345" rpy="${-pi/2} 0 ${-pi/2}"/>
+  <parent link="$(arg robot_name)/gripper_link"/>
+  <child link="$(arg robot_name)/led_link1"/> </joint>
+<link name="$(arg robot_name)/led_link1">
+  </link>
+    <gazebo reference="$(arg robot_name)/gripper_link">
+    <sensor type="depth" name="depth_camera">
+    <pose>0.06645 0 0.043 0 0 0</pose>
+      <update_rate>10</update_rate>
+      <camera>
+        <horizontal_fov>${pi/6}</horizontal_fov>
+        <image>
+          <width>640</width>
+          <height>480</height>
+          <format>R8G8B8</format>
+        </image>
+        <clip>
+          <near>0.02</near>
+          <far>1</far>
+        </clip>
+      </camera>
+          <plugin name="camera_plugin" filename="libgazebo_ros_openni_kinect.so">
+          <baseline>0.2</baseline>
+          <alwaysOn>true</alwaysOn>
+          <!-- Keep this zero, update_rate in the parent <sensor> tag
+            will control the frame rate. -->
+          <updateRate>0.0</updateRate>
+          <cameraName>depth_camera</cameraName>
+          <imageTopicName>/depth_camera/color/image_raw</imageTopicName>
+          <cameraInfoTopicName>/depth_camera/color/camera_info</cameraInfoTopicName>
+          <depthImageTopicName>/depth_camera/depth/image_raw</depthImageTopicName>
+          <depthImageCameraInfoTopicName>/depth_camera/depth/camera_info</depthImageCameraInfoTopicName>
+          <pointCloudTopicName>/depth_camera/depth/points</pointCloudTopicName>
+          <frameName>odom</frameName>
+          <pointCloudCutoff>0.0</pointCloudCutoff>
+          <pointCloudCutoffMax>1.0</pointCloudCutoffMax>
+          <distortionK1>0</distortionK1>
+          <distortionK2>0</distortionK2>
+          <distortionK3>0</distortionK3>
+          <distortionT1>0</distortionT1>
+          <distortionT2>0</distortionT2>
+          <CxPrime>0</CxPrime>
+          <Cx>0</Cx>
+          <Cy>0</Cy>
+          <focalLength>0</focalLength>
+          <hackBaseline>0</hackBaseline>
+        </plugin>
+    </sensor>
+  </gazebo>
   <gazebo reference="$(arg robot_name)/gripper_link">
   <light name ='led' type = 'spot'>

Commit message: Added lights to the additional nozzles
Added lights to the additional nozzles which are controlled by the same spray commmand message as original

File: ros-workspace/src/dr_phil_description/urdf/px100.urdf.xacro (robot description, xacro)
@@ -447,4 +447,44 @@
         </inertial>
       </link>
+      <joint name="$(arg robot_name)/led_left_joint" type="fixed">
+  <origin xyz="0.029 0.021 0.01248" rpy="0 0 ${-pi/6}"/>
+  <parent link="$(arg robot_name)/left_finger_link"/>
+  <child link="$(arg robot_name)/led_left_link"/> </joint>
+<link name="$(arg robot_name)/led_left_link">
+   <visual>
+      <origin rpy="0 0 0" xyz="0 0.0 0.0"/>
+      <geometry>
+        <mesh filename="package://dr_phil_description/meshes/spray_components/8_5mm_nozzle.stl" scale="0.001 0.001 0.001"/>
+      </geometry>
+      <material name="black"/>
+    </visual>
+   <collision>
+      <origin rpy="0 0 0" xyz="0 0 0"/>
+      <geometry>
+        <mesh filename="package://dr_phil_description/meshes/spray_components/8_5mm_nozzle.stl" scale="0.001 0.001 0.001"/>
+      </geometry>
+    </collision>
+    <inertial>
+      <origin rpy="0 0 0" xyz="0 0 0"/>
+      <mass value="0.002" />
+      <inertia ixx="0.00" iyy="0.00" izz="0.000" ixy="0.0000000000" ixz="0.0000000000" iyz="0" />
+    </inertial>
+  </link>
+  <gazebo reference="$(arg robot_name)/left_finger_link">
+  <light name ='led' type = 'spot'>
+    <pose>0.0392 -0.007 0.021 0 ${-pi/2} ${-pi/6}</pose><!--you can place light position here ,and it is useless to give position in link-->
+    <attenuation>
+            <range>0</range>
+          </attenuation>
+          <diffuse>1 1 1 0</diffuse>
+          <specular>1 1 1 0</specular>
+          <spot>
+            <inner_angle>${pi/6}</inner_angle>
+            <outer_angle>${pi/6}</outer_angle>
+            <falloff>1</falloff>
+          </spot>
+          <cast_shadows>1</cast_shadows>
+  </light>
+  </gazebo>
       <joint name="gripper_sub" type="prismatic">
         <axis xyz="0 1 0"/>
@@ -485,4 +525,44 @@
         </inertial>
       </link>
+      <joint name="$(arg robot_name)/led_right_joint" type="fixed">
+  <origin xyz="0.01 0.012 0.01248" rpy="0 0 ${pi/6}"/>
+  <parent link="$(arg robot_name)/right_finger_link"/>
+  <child link="$(arg robot_name)/led_right_link"/> </joint>
+<link name="$(arg robot_name)/led_right_link">
+   <visual>
+      <origin rpy="0 0 0" xyz="0 0.0 0.0"/>
+      <geometry>
+        <mesh filename="package://dr_phil_description/meshes/spray_components/8_5mm_nozzle.stl" scale="0.001 0.001 0.001"/>
+      </geometry>
+      <material name="black"/>
+    </visual>
+   <collision>
+      <origin rpy="0 0 0" xyz="0 0 0"/>
+      <geometry>
+        <mesh filename="package://dr_phil_description/meshes/spray_components/8_5mm_nozzle.stl" scale="0.001 0.001 0.001"/>
+      </geometry>
+    </collision>
+    <inertial>
+      <origin rpy="0 0 0" xyz="0 0 0"/>
+      <mass value="0.002" />
+      <inertia ixx="0.00" iyy="0.00" izz="0.000" ixy="0.0000000000" ixz="0.0000000000" iyz="0" />
+    </inertial>
+  </link>
+<gazebo reference="$(arg robot_name)/right_finger_link">
+  <light name ='led' type = 'spot'>
+    <pose>0.0394 0.007 0.021 0 ${-pi/2} ${pi/6}</pose><!--you can place light position here ,and it is useless to give position in link-->
+    <attenuation>
+            <range>0</range>
+          </attenuation>
+          <diffuse>1 1 1 0</diffuse>
+          <specular>1 1 1 0</specular>
+          <spot>
+            <inner_angle>${pi/6}</inner_angle>
+            <outer_angle>${pi/6}</outer_angle>
+            <falloff>1</falloff>
+          </spot>
+          <cast_shadows>1</cast_shadows>
+  </light>
+  </gazebo>
       <joint name="ee_gripper" type="fixed">
         <axis xyz="1 0 0"/>

Commit message: added coverage of additional nozzles

File: ros-workspace/src/dr_phil_description/urdf/px100.urdf.xacro (robot description, xacro)
@@ -252,6 +252,6 @@
     <gazebo reference="$(arg robot_name)/gripper_link">
     <sensor type="depth" name="depth_camera">
-    <pose>0.06645 0 0.043 0 0 0</pose>
-      <update_rate>20</update_rate>
+    <pose>0.044 0.019 0.0345 0 0 0</pose>
+      <update_rate>4</update_rate>
       <camera>
         <horizontal_fov>${pi/6}</horizontal_fov>
@@ -279,5 +279,5 @@
           <pointCloudTopicName>/depth_camera/depth/points</pointCloudTopicName>
           <frameName>$(arg robot_name)/led_link1</frameName>
-          <pointCloudCutoff>0.0</pointCloudCutoff>
+          <pointCloudCutoff>0.095</pointCloudCutoff>
           <pointCloudCutoffMax>1.0</pointCloudCutoffMax>
           <distortionK1>0</distortionK1>
@@ -471,4 +471,54 @@
     </inertial>
   </link>
+  <joint name="$(arg robot_name)/led_left_joint1" type="fixed">
+  <origin xyz="0.029 0.021 0.01248" rpy="${-pi/2} 0 ${(-pi/2)}"/>
+  <parent link="$(arg robot_name)/left_finger_link"/>
+  <child link="$(arg robot_name)/led_left_link1"/> </joint>
+<link name="$(arg robot_name)/led_left_link1">
+  </link>
+  <gazebo reference="$(arg robot_name)/left_finger_link">
+    <sensor type="depth" name="depth_left">
+    <pose>0.029 0.021 0.012480  0 0</pose>
+      <update_rate>4</update_rate>
+      <camera>
+        <horizontal_fov>${pi/6}</horizontal_fov>
+        <image>
+          <width>640</width>
+          <height>480</height>
+          <format>R8G8B8</format>
+        </image>
+        <clip>
+          <near>0.02</near>
+          <far>1</far>
+        </clip>
+      </camera>
+          <plugin name="camera_plugin" filename="libgazebo_ros_openni_kinect.so">
+          <baseline>0.2</baseline>
+          <alwaysOn>true</alwaysOn>
+          <!-- Keep this zero, update_rate in the parent <sensor> tag
+            will control the frame rate. -->
+          <updateRate>0.0</updateRate>
+          <cameraName>depth_left</cameraName>
+          <imageTopicName>/depth_left/color/image_raw</imageTopicName>
+          <cameraInfoTopicName>/depth_left/color/camera_info</cameraInfoTopicName>
+          <depthImageTopicName>/depth_left/depth/image_raw</depthImageTopicName>
+          <depthImageCameraInfoTopicName>/depth_left/depth/camera_info</depthImageCameraInfoTopicName>
+          <pointCloudTopicName>/depth_left/depth/points</pointCloudTopicName>
+          <frameName>$(arg robot_name)/led_left_link1</frameName>
+          <pointCloudCutoff>0.06</pointCloudCutoff>
+          <pointCloudCutoffMax>1.0</pointCloudCutoffMax>
+          <distortionK1>0</distortionK1>
+          <distortionK2>0</distortionK2>
+          <distortionK3>0</distortionK3>
+          <distortionT1>0</distortionT1>
+          <distortionT2>0</distortionT2>
+          <CxPrime>0</CxPrime>
+          <Cx>0</Cx>
+          <Cy>0</Cy>
+          <focalLength>0</focalLength>
+          <hackBaseline>0</hackBaseline>
+        </plugin>
+    </sensor>
+  </gazebo>
   <gazebo reference="$(arg robot_name)/left_finger_link">
   <light name ='led' type = 'spot'>
@@ -549,4 +599,54 @@
     </inertial>
   </link>
+  <joint name="$(arg robot_name)/led_right_joint1" type="fixed">
+  <origin xyz="0.01 0.012 0.01248" rpy="${-pi/2} 0 ${-pi/2}"/>
+  <parent link="$(arg robot_name)/right_finger_link"/>
+  <child link="$(arg robot_name)/led_right_link1"/> </joint>
+<link name="$(arg robot_name)/led_right_link1">
+  </link>
+  <gazebo reference="$(arg robot_name)/right_finger_link">
+    <sensor type="depth" name="depth_right">
+    <pose>0.01 0.012 0.01248 0  0 0</pose>
+      <update_rate>4</update_rate>
+      <camera>
+        <horizontal_fov>${pi/6}</horizontal_fov>
+        <image>
+          <width>640</width>
+          <height>480</height>
+          <format>R8G8B8</format>
+        </image>
+        <clip>
+          <near>0.02</near>
+          <far>1</far>
+        </clip>
+      </camera>
+          <plugin name="camera_plugin" filename="libgazebo_ros_openni_kinect.so">
+          <baseline>0.2</baseline>
+          <alwaysOn>true</alwaysOn>
+          <!-- Keep this zero, update_rate in the parent <sensor> tag
+            will control the frame rate. -->
+          <updateRate>0.0</updateRate>
+          <cameraName>depth_right</cameraName>
+          <imageTopicName>/depth_right/color/image_raw</imageTopicName>
+          <cameraInfoTopicName>/depth_right/color/camera_info</cameraInfoTopicName>
+          <depthImageTopicName>/depth_right/depth/image_raw</depthImageTopicName>
+          <depthImageCameraInfoTopicName>/depth_right/depth/camera_info</depthImageCameraInfoTopicName>
+          <pointCloudTopicName>/depth_right/depth/points</pointCloudTopicName>
+          <frameName>$(arg robot_name)/led_right_link1</frameName>
+          <pointCloudCutoff>0.06</pointCloudCutoff>
+          <pointCloudCutoffMax>1.0</pointCloudCutoffMax>
+          <distortionK1>0</distortionK1>
+          <distortionK2>0</distortionK2>
+          <distortionK3>0</distortionK3>
+          <distortionT1>0</distortionT1>
+          <distortionT2>0</distortionT2>
+          <CxPrime>0</CxPrime>
+          <Cx>0</Cx>
+          <Cy>0</Cy>
+          <focalLength>0</focalLength>
+          <hackBaseline>0</hackBaseline>
+        </plugin>
+    </sensor>
+  </gazebo>
 <gazebo reference="$(arg robot_name)/right_finger_link">
   <light name ='led' type = 'spot'>
