Commit message: Fixed model breaking arm movement

File: ros-workspace/src/dr_phil_description/urdf/px100.urdf.xacro (robot description, xacro)
@@ -232,15 +232,4 @@
       <material name="black"/>
     </visual>
-   <collision>
-      <origin rpy="0 0 0" xyz="0 0 0"/>
-      <geometry>
-        <mesh filename="package://dr_phil_description/meshes/spray_components/8_5mm_nozzle.stl" scale="0.001 0.001 0.001"/>
-      </geometry>
-    </collision>
-    <inertial>
-      <origin rpy="0 0 0" xyz="0 0 0"/>
-      <mass value="0.002" />
-      <inertia ixx="0.00" iyy="0.00" izz="0.000" ixy="0.0000000000" ixz="0.0000000000" iyz="0" />
-    </inertial>
   </link>
     <joint name="$(arg robot_name)/led_joint1" type="fixed">
@@ -253,5 +242,5 @@
     <sensor type="depth" name="depth_camera">
     <pose>0.044 0.019 0.0345 0 0 0</pose>
-      <update_rate>4</update_rate>
+      <update_rate>20</update_rate>
       <camera>
         <horizontal_fov>${pi/6}</horizontal_fov>
@@ -459,15 +448,4 @@
       <material name="black"/>
     </visual>
-   <collision>
-      <origin rpy="0 0 0" xyz="0 0 0"/>
-      <geometry>
-        <mesh filename="package://dr_phil_description/meshes/spray_components/8_5mm_nozzle.stl" scale="0.001 0.001 0.001"/>
-      </geometry>
-    </collision>
-    <inertial>
-      <origin rpy="0 0 0" xyz="0 0 0"/>
-      <mass value="0.002" />
-      <inertia ixx="0.00" iyy="0.00" izz="0.000" ixy="0.0000000000" ixz="0.0000000000" iyz="0" />
-    </inertial>
   </link>
   <joint name="$(arg robot_name)/led_left_joint1" type="fixed">
@@ -480,5 +458,5 @@
     <sensor type="depth" name="depth_left">
     <pose>0.029 0.021 0.012480  0 0</pose>
-      <update_rate>4</update_rate>
+      <update_rate>20</update_rate>
       <camera>
         <horizontal_fov>${pi/6}</horizontal_fov>
@@ -587,15 +565,4 @@
       <material name="black"/>
     </visual>
-   <collision>
-      <origin rpy="0 0 0" xyz="0 0 0"/>
-      <geometry>
-        <mesh filename="package://dr_phil_description/meshes/spray_components/8_5mm_nozzle.stl" scale="0.001 0.001 0.001"/>
-      </geometry>
-    </collision>
-    <inertial>
-      <origin rpy="0 0 0" xyz="0 0 0"/>
-      <mass value="0.002" />
-      <inertia ixx="0.00" iyy="0.00" izz="0.000" ixy="0.0000000000" ixz="0.0000000000" iyz="0" />
-    </inertial>
   </link>
   <joint name="$(arg robot_name)/led_right_joint1" type="fixed">
@@ -608,5 +575,5 @@
     <sensor type="depth" name="depth_right">
     <pose>0.01 0.012 0.01248 0  0 0</pose>
-      <update_rate>4</update_rate>
+      <update_rate>20</update_rate>
       <camera>
         <horizontal_fov>${pi/6}</horizontal_fov>

Commit message: changed nozzle angle

File: ros-workspace/src/dr_phil_description/urdf/px100.urdf.xacro (robot description, xacro)
@@ -437,5 +437,5 @@
       </link>
       <joint name="$(arg robot_name)/led_left_joint" type="fixed">
-  <origin xyz="0.029 0.021 0.01248" rpy="0 0 ${-pi/6}"/>
+  <origin xyz="0.108 0.012 0.01248" rpy="0 0 ${-pi/2}"/>
   <parent link="$(arg robot_name)/left_finger_link"/>
   <child link="$(arg robot_name)/led_left_link"/> </joint>
@@ -450,5 +450,5 @@
   </link>
   <joint name="$(arg robot_name)/led_left_joint1" type="fixed">
-  <origin xyz="0.029 0.021 0.01248" rpy="${-pi/2} 0 ${(-pi/2)}"/>
+  <origin xyz="0.108 0.012 0.01248" rpy="${-pi/2} 0 ${(-pi/2)-pi/2}"/>
   <parent link="$(arg robot_name)/left_finger_link"/>
   <child link="$(arg robot_name)/led_left_link1"/> </joint>
@@ -457,5 +457,5 @@
   <gazebo reference="$(arg robot_name)/left_finger_link">
     <sensor type="depth" name="depth_left">
-    <pose>0.029 0.021 0.012480  0 0</pose>
+    <pose>0.108 0.012 0.01248 0  0 ${-pi/2}</pose>
       <update_rate>20</update_rate>
       <camera>
@@ -484,5 +484,5 @@
           <pointCloudTopicName>/depth_left/depth/points</pointCloudTopicName>
           <frameName>$(arg robot_name)/led_left_link1</frameName>
-          <pointCloudCutoff>0.06</pointCloudCutoff>
+          <pointCloudCutoff>0.02</pointCloudCutoff>
           <pointCloudCutoffMax>1.0</pointCloudCutoffMax>
           <distortionK1>0</distortionK1>
@@ -501,5 +501,5 @@
   <gazebo reference="$(arg robot_name)/left_finger_link">
   <light name ='led' type = 'spot'>
-    <pose>0.0392 -0.007 0.021 0 ${-pi/2} ${-pi/6}</pose><!--you can place light position here ,and it is useless to give position in link-->
+    <pose>0.088 -0.007 0.021 0 ${-pi/2} ${-pi/2}</pose><!--you can place light position here ,and it is useless to give position in link-->
     <attenuation>
             <range>0</range>
@@ -554,5 +554,5 @@
       </link>
       <joint name="$(arg robot_name)/led_right_joint" type="fixed">
-  <origin xyz="0.01 0.012 0.01248" rpy="0 0 ${pi/6}"/>
+  <origin xyz="0.07 -0.012 0.01248" rpy="0 0 ${pi/2}"/>
   <parent link="$(arg robot_name)/right_finger_link"/>
   <child link="$(arg robot_name)/led_right_link"/> </joint>
@@ -567,5 +567,5 @@
   </link>
   <joint name="$(arg robot_name)/led_right_joint1" type="fixed">
-  <origin xyz="0.01 0.012 0.01248" rpy="${-pi/2} 0 ${-pi/2}"/>
+  <origin xyz="0.7 -0.012 0.01248" rpy="${-pi/2} 0 ${(pi/2)-pi/2}"/>
   <parent link="$(arg robot_name)/right_finger_link"/>
   <child link="$(arg robot_name)/led_right_link1"/> </joint>
@@ -574,5 +574,5 @@
   <gazebo reference="$(arg robot_name)/right_finger_link">
     <sensor type="depth" name="depth_right">
-    <pose>0.01 0.012 0.01248 0  0 0</pose>
+    <pose>0.7 -0.012 0.01248 0  0 ${(pi/2)}</pose>
       <update_rate>20</update_rate>
       <camera>
@@ -618,5 +618,5 @@
 <gazebo reference="$(arg robot_name)/right_finger_link">
   <light name ='led' type = 'spot'>
-    <pose>0.0394 0.007 0.021 0 ${-pi/2} ${pi/6}</pose><!--you can place light position here ,and it is useless to give position in link-->
+    <pose>0.0882 0.007 0.021 0 ${-pi/2} ${pi/2}</pose><!--you can place light position here ,and it is useless to give position in link-->
     <attenuation>
             <range>0</range>

Commit message: nozzle change

File: ros-workspace/src/dr_phil_description/urdf/px100.urdf.xacro (robot description, xacro)
@@ -437,5 +437,5 @@
       </link>
       <joint name="$(arg robot_name)/led_left_joint" type="fixed">
-  <origin xyz="0.108 0.012 0.01248" rpy="0 0 ${-pi/2}"/>
+  <origin xyz="0.108 0.055 0.01248" rpy="0 0 ${-pi/2}"/>
   <parent link="$(arg robot_name)/left_finger_link"/>
   <child link="$(arg robot_name)/led_left_link"/> </joint>
@@ -450,5 +450,5 @@
   </link>
   <joint name="$(arg robot_name)/led_left_joint1" type="fixed">
-  <origin xyz="0.108 0.012 0.01248" rpy="${-pi/2} 0 ${(-pi/2)-pi/2}"/>
+  <origin xyz="0.108 0.055 0.01248" rpy="${-pi/2} 0 ${(-pi/2)-pi/2}"/>
   <parent link="$(arg robot_name)/left_finger_link"/>
   <child link="$(arg robot_name)/led_left_link1"/> </joint>
@@ -457,5 +457,5 @@
   <gazebo reference="$(arg robot_name)/left_finger_link">
     <sensor type="depth" name="depth_left">
-    <pose>0.108 0.012 0.01248 0  0 ${-pi/2}</pose>
+    <pose>0.108 0.055 0.01248 0  0 ${-pi/2}</pose>
       <update_rate>20</update_rate>
       <camera>
@@ -484,5 +484,5 @@
           <pointCloudTopicName>/depth_left/depth/points</pointCloudTopicName>
           <frameName>$(arg robot_name)/led_left_link1</frameName>
-          <pointCloudCutoff>0.02</pointCloudCutoff>
+          <pointCloudCutoff>0.0</pointCloudCutoff>
           <pointCloudCutoffMax>1.0</pointCloudCutoffMax>
           <distortionK1>0</distortionK1>
@@ -501,5 +501,5 @@
   <gazebo reference="$(arg robot_name)/left_finger_link">
   <light name ='led' type = 'spot'>
-    <pose>0.088 -0.007 0.021 0 ${-pi/2} ${-pi/2}</pose><!--you can place light position here ,and it is useless to give position in link-->
+    <pose>0.088 0.045 0.021 0 ${-pi/2} ${-pi/2}</pose><!--you can place light position here ,and it is useless to give position in link-->
     <attenuation>
             <range>0</range>
@@ -554,5 +554,5 @@
       </link>
       <joint name="$(arg robot_name)/led_right_joint" type="fixed">
-  <origin xyz="0.07 -0.012 0.01248" rpy="0 0 ${pi/2}"/>
+  <origin xyz="0.07 -0.055 0.01248" rpy="0 0 ${pi/2}"/>
   <parent link="$(arg robot_name)/right_finger_link"/>
   <child link="$(arg robot_name)/led_right_link"/> </joint>
@@ -567,5 +567,5 @@
   </link>
   <joint name="$(arg robot_name)/led_right_joint1" type="fixed">
-  <origin xyz="0.7 -0.012 0.01248" rpy="${-pi/2} 0 ${(pi/2)-pi/2}"/>
+  <origin xyz="0.7 -0.055 0.01248" rpy="${-pi/2} 0 ${(pi/2)-pi/2}"/>
   <parent link="$(arg robot_name)/right_finger_link"/>
   <child link="$(arg robot_name)/led_right_link1"/> </joint>
@@ -574,5 +574,5 @@
   <gazebo reference="$(arg robot_name)/right_finger_link">
     <sensor type="depth" name="depth_right">
-    <pose>0.7 -0.012 0.01248 0  0 ${(pi/2)}</pose>
+    <pose>0.7 -0.055 0.01248 0  0 ${(pi/2)}</pose>
       <update_rate>20</update_rate>
       <camera>
@@ -601,5 +601,5 @@
           <pointCloudTopicName>/depth_right/depth/points</pointCloudTopicName>
           <frameName>$(arg robot_name)/led_right_link1</frameName>
-          <pointCloudCutoff>0.06</pointCloudCutoff>
+          <pointCloudCutoff>0.0</pointCloudCutoff>
           <pointCloudCutoffMax>1.0</pointCloudCutoffMax>
           <distortionK1>0</distortionK1>
@@ -618,5 +618,5 @@
 <gazebo reference="$(arg robot_name)/right_finger_link">
   <light name ='led' type = 'spot'>
-    <pose>0.0882 0.007 0.021 0 ${-pi/2} ${pi/2}</pose><!--you can place light position here ,and it is useless to give position in link-->
+    <pose>0.0882 -0.05 0.021 0 ${-pi/2} ${pi/2}</pose><!--you can place light position here ,and it is useless to give position in link-->
     <attenuation>
             <range>0</range>

Commit message: nozzles update

File: ros-workspace/src/dr_phil_description/urdf/px100.urdf.xacro (robot description, xacro)
@@ -567,5 +567,5 @@
   </link>
   <joint name="$(arg robot_name)/led_right_joint1" type="fixed">
-  <origin xyz="0.7 -0.055 0.01248" rpy="${-pi/2} 0 ${(pi/2)-pi/2}"/>
+  <origin xyz="0.07 -0.055 0.01248" rpy="${-pi/2} 0 ${(pi/2)-pi/2}"/>
   <parent link="$(arg robot_name)/right_finger_link"/>
   <child link="$(arg robot_name)/led_right_link1"/> </joint>
@@ -574,5 +574,5 @@
   <gazebo reference="$(arg robot_name)/right_finger_link">
     <sensor type="depth" name="depth_right">
-    <pose>0.7 -0.055 0.01248 0  0 ${(pi/2)}</pose>
+    <pose>0.07 -0.055 0.01248 0  0 ${(pi/2)}</pose>
       <update_rate>20</update_rate>
       <camera>

Commit message: adjusted robot properties for door opening

File: ros-workspace/src/dr_phil_description/urdf/px100.urdf.xacro (robot description, xacro)
@@ -429,4 +429,18 @@
             <mesh filename="package://dr_phil_description/meshes/px100_meshes/px100_8_gripper_finger.stl" scale="0.001 0.001 0.001"/>
           </geometry>
+            <surface>
+            <friction>
+              <ode>
+                <mu>1</mu>
+                <mu2>1</mu2>
+              </ode>
+            </friction>
+          </surface>
+        </collision>
+        <collision>
+            <origin rpy="${pi} ${pi} 0" xyz="0.045 -0.01 0"/>
+          <geometry>
+           <cylinder length="0.030" radius="0.003"/>
+          </geometry>
         </collision>
         <inertial>
@@ -533,4 +547,36 @@
         </actuator>
       </transmission>
+      <gazebo reference="$(arg robot_name)/right_finger_link">
+        <mu1>1000</mu1>
+        <mu2>1000</mu2>
+        <kp>1000000.0</kp>
+        <kd>100000.0</kd>
+        <slip1>0</slip1>
+        <slip2>0</slip2>
+        <minDepth>0.001</minDepth>
+        <maxVel>0</maxVel>
+        <torsional>
+          <ode>
+              <coefficient>1000</coefficient>
+              <slip>0</slip>
+          </ode>
+        </torsional>
+      </gazebo>
+      <gazebo reference="$(arg robot_name)/left_finger_link">
+        <mu1>1000</mu1>
+        <mu2>1000</mu2>
+        <kp>1000000.0</kp>
+        <kd>100000.0</kd>
+        <slip1>0</slip1>
+        <slip2>0</slip2>
+        <minDepth>0.001</minDepth>
+        <maxVel>0</maxVel>
+        <torsional>
+          <ode>
+              <coefficient>1000</coefficient>
+              <slip>0</slip>
+          </ode>
+        </torsional>
+      </gazebo>
       <link name="$(arg robot_name)/right_finger_link">
         <visual>
@@ -545,4 +591,16 @@
           <geometry>
             <mesh filename="package://dr_phil_description/meshes/px100_meshes/px100_8_gripper_finger.stl" scale="0.001 0.001 0.001"/>
+          </geometry>
+            <friction>
+              <ode>
+                <mu>1</mu>
+                <mu2>1</mu2>
+              </ode>
+            </friction>
+        </collision>
+        <collision>
+            <origin rpy="${pi} ${pi} 0" xyz="0.045 0.01 0"/>
+          <geometry>
+           <cylinder length="0.030" radius="0.003"/>
           </geometry>
         </collision>
